File: pc1715-esp32vga/pc1715-esp32vga.kicad_sch (KiCad schematic)
At the start: 38 parts, among them J1 IDC10_VIDEO_IN, J2 VGAOUT, J3 USB_B, J4 KEYPAD, J5 IDC16_VGAOUT, J6 USB_C_Receptacle_USB2.0_16P, J7 DBG, J8 EXT-5V, U1 LM1117MP-3.3, U2 ESP32-S3-WROOM-1

Commit message: add part order numbers for Reichelt and JLCPCB (allow PCBA)
Parts:
- C1: JLCPCB Part # (none) -> C308881; Reichelt (none) -> TPS 3225 47/10
- C2: JLCPCB Part # (none) -> C74423; Reichelt (none) -> TPS 3216 10/10
- D1: JLCPCB Part # (none) -> MHT170CRCT
- D4, D5, D6: JLCPCB Part # (none) -> C77356; Reichelt (none) -> SD103BW DIO
- J6: JLCPCB Part # (none) -> C5184243
- R1: JLCPCB Part # (none) -> C17414; Reichelt (none) -> SMD-0805 10,0K
- R10, R6, R8: JLCPCB Part # (none) -> C17710; Reichelt (none) -> SMD-0805 470
- R11, R12, R13, R2, R3, R4: JLCPCB Part # (none) -> C17630; Reichelt (none) -> PAN ERJ6ENF3300V
- R5, R7, R9: JLCPCB Part # (none) -> C441981; Reichelt (none) -> PAN ERJP06F1001
- U1: JLCPCB Part # (none) -> C9662; Reichelt (none) -> LM 1117 MPX-3.3
- U2: JLCPCB Part # (none) -> C2913201; Reichelt (none) -> ESP32S3WRM1N8R8
